File: hardware/CANpaca-EB-schematics/CANpaca-EB-schematics.kicad_pcb (KiCad board)
At the start: 4 copper layers, 42 x 42 mm, 132 parts, among them J11 Conn_01x03_Male, J12 A2501WV-4P, J13 A2501WV-3P, J14 A2501WV-5P, J16 A2501WV-3P, J17 A2501WV-2P, J2 FAN_0, J4 Conn_01x03_Male, J5 FAN_1, J6 Screw_Terminal_01x02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

Commit message: added schematic pdf
Changed lines of the file:
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@@
       (outputformat 1)
       (mirror false)
-      (drillshape 1)
+      (drillshape 0)
       (scaleselection 1)
-      (outputdirectory "")
+      (outputdirectory "gerber/")
     )
   )
@@
     (fp_line (start -3.5 -2.5) (end -2.5 -3.5) (layer "F.Fab") (width 0.1))
     (fp_line (start -3.5 3.5) (end -3.5 -2.5) (layer "F.Fab") (width 0.1))
-    (pad "" smd roundrect locked (at 0.8 0.8) (size 1.29 1.29) (layers "F.Paste") (roundrect_rratio 0.193798))
-    (pad "" smd roundrect locked (at 0.8 -0.8) (size 1.29 1.29) (layers "F.Paste") (roundrect_rratio 0.193798))
-    (pad "" smd roundrect locked (at -0.8 0.8) (size 1.29 1.29) (layers "F.Paste") (roundrect_rratio 0.193798))
-    (pad "" smd roundrect locked (at -0.8 -0.8) (size 1.29 1.29) (layers "F.Paste") (roundrect_rratio 0.193798))
+    (pad "" smd roundrect locked (at 0.8 0.8) (size 1.29 1.29) (layers "F.Paste") (roundrect_rratio 0.1937976744))
+    (pad "" smd roundrect locked (at 0.8 -0.8) (size 1.29 1.29) (layers "F.Paste") (roundrect_rratio 0.1937976744))
+    (pad "" smd roundrect locked (at -0.8 0.8) (size 1.29 1.29) (layers "F.Paste") (roundrect_rratio 0.1937976744))
+    (pad "" smd roundrect locked (at -0.8 -0.8) (size 1.29 1.29) (layers "F.Paste") (roundrect_rratio 0.1937976744))
     (pad "1" smd roundrect locked (at -3.4375 -2.6) (size 0.875 0.2) (layers "F.Cu" "F.Paste" "F.Mask") (roundrect_rratio 0.25)
       (net 10 "3V3") (pinfunction "IOVDD") (pintype "power_in"))
@@
     (fp_line (start 6.575 -7.92) (end 6.575 0.99) (layer "F.Fab") (width 0.1))
     (pad "" np_thru_hole circle (at 1.5 -4.32) (size 3 3) (drill 3) (layers *.Cu *.Mask))
-    (pad "1" thru_hole roundrect (at 0 0) (size 1.5 1.5) (drill 1.02) (layers *.Cu *.Mask) (roundrect_rratio 0.166667)
+    (pad "1" thru_hole roundrect (at 0 0) (size 1.5 1.5) (drill 1.02) (layers *.Cu *.Mask) (roundrect_rratio 0.1666673333)
       (net 6 "DC_IN") (pinfunction "Pin_1") (pintype "passive"))
     (pad "2" thru_hole circle (at 3 0) (size 1.5 1.5) (drill 1.02) (layers *.Cu *.Mask)
@@
     (fp_line (start -2.5 1.5) (end -1.5 2.5) (layer "B.Fab") (width 0.1))
     (fp_line (start 2.5 -2.5) (end -2.5 -2.5) (layer "B.Fab") (width 0.1))
-    (pad "" smd roundrect (at -0.81 -0.81 180) (size 1.31 1.31) (layers "B.Paste") (roundrect_rratio 0.19084))
-    (pad "" smd roundrect (at -0.81 0.81 180) (size 1.31 1.31) (layers "B.Paste") (roundrect_rratio 0.19084))
-    (pad "" smd roundrect (at 0.81 -0.81 180) (size 1.31 1.31) (layers "B.Paste") (roundrect_rratio 0.19084))
-    (pad "" smd roundrect (at 0.81 0.81 180) (size 1.31 1.31) (layers "B.Paste") (roundrect_rratio 0.19084))
+    (pad "" smd roundrect (at -0.81 -0.81 180) (size 1.31 1.31) (layers "B.Paste") (roundrect_rratio 0.1908396947))
+    (pad "" smd roundrect (at -0.81 0.81 180) (size 1.31 1.31) (layers "B.Paste") (roundrect_rratio 0.1908396947))
+    (pad "" smd roundrect (at 0.81 -0.81 180) (size 1.31 1.31) (layers "B.Paste") (roundrect_rratio 0.1908396947))
+    (pad "" smd roundrect (at 0.81 0.81 180) (size 1.31 1.31) (layers "B.Paste") (roundrect_rratio 0.1908396947))
     (pad "1" smd roundrect (at -2.4375 1.3 180) (size 0.825 0.3) (layers "B.Cu" "B.Paste" "B.Mask") (roundrect_rratio 0.25)
       (net 74 "Net-(R26-Pad2)") (pinfunction "BIAS") (pintype "power_out"))

Commit message: fixed usb resistor
Parts:
- R18, R23: value 22R -> 27R
Changed lines of the file:
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@@
       (effects (font (size 1 1) (thickness 0.15)))
     )
-    (fp_text value "22R" (at 0 1.43 90) (layer "F.Fab") hide
+    (fp_text value "27R" (at 0 1.43 90) (layer "F.Fab") hide
       (effects (font (size 1 1) (thickness 0.15)))
     )
@@
       (effects (font (size 1 1) (thickness 0.15)))
     )
-    (fp_text value "22R" (at 0 1.43 90) (layer "F.Fab") hide
+    (fp_text value "27R" (at 0 1.43 90) (layer "F.Fab") hide
       (effects (font (size 1 1) (thickness 0.15)))
     )
